File: CPU1-NRF5340-uBlox-NORA.kicad_pcb (KiCad board)
At the start: 6 copper layers, 50 x 30 mm, 75 parts, among them CON1 FH12-12S-0.5SVA_54_, CON2 FH12-12S-0.5SVA_54_, CON3 FH12-12S-0.5SVA_54_, CON4 FH12-12S-0.5SVA_54_, J1 U262-161N-4BVC11, J4 S2B-PH-SM4-TB, J5 Conn_01x08_MountingPin, Q1 BSS123, SW1 SW_SPST_ALPS_SKSCLDE010, SW2 SW_SPST_ALPS_SKSCLDE010, U2 ADC081C021CIMM, U3 PCA9557BS, U4 74HC4051BQ, U5 RT6154AGQW, U6 MCP73831T-2DCI/OT, U7 TPS2116DRL, U8 NORA-B106-00B, Y1 Crystal

Commit message: files after sent to Bittele, with corrections for Bittele
Parts:
- removed the D3 at (113.5, 104.0)
- added D4: EASV3015RGBA0, Zed-Library:LED_RGB_Everlight_EASV3015RGBA0_Horizontal, F.Cu at (113.9, 103.5)
- D1: renamed from D2; value RB161QS-40 -> SBR0240LPW-7B
- J1: value U262-161N-4BVC11 -> GCT USB4105; footprint Connector_USB:USB_C_Receptacle_XKB_U262-16XN-4BVC11 -> Connector_USB:USB_C_Receptacle_GCT_USB4105-xx-A_16P_TopMnt_Horizontal
- J2: renamed from J5; value Conn_01x08_MountingPin -> FH12-8S-0.5SH; footprint Zed-Library:XunPu_FPC-05FB-8PH20_01x08_P0.5mm_Horizontal -> Connector_FFC-FPC:Hirose_FH12-8S-0.5SH_1x08-1MP_P0.50mm_Horizontal
- J3: renamed from J4; footprint LJK_Library:JST_PH_S2B-PH-SM4-TB_1x02-1MP_P2.00mm_Horizontal -> Zed-Library:JST_PH_S2B-PH-SM4-TB_1x02-1MP_P2.00mm_Horizontal
- R25: renamed from R14; value 100 -> 39
- R26: renamed from R12; value 100 -> 130
- R27: renamed from R13; value 100 -> 30
- U2: renamed from U3; footprint Package_DFN_QFN:HVQFN-16-1EP_3x3mm_P0.5mm_EP1.5x1.5mm -> Package_DFN_QFN:Texas_RGV0016A_VQFN-16-1EP_4x4mm_P0.65mm_EP2.1x2.1mm
- moved C15 6.05 mm to (130.6, 97.7)
- moved J2 1.81 mm to (124.3, 99.8)
- moved C3 1.63 mm to (123.7, 81.0)
- moved U2 0.60 mm to (120.0, 81.1)
- moved R26 0.51 mm to (115.0, 100.7)
- moved R25 0.50 mm to (113.0, 100.7)
- moved R27 0.50 mm to (114.0, 100.7)
- moved C2 0.25 mm to (113.7, 78.2)
- moved J1 0.12 mm to (151.8, 86.0)
- renumbered C16 to C1, C15 to C10, C3 to C11, C8 to C12, C5 to C13, C9 to C14, C6 to C15, C10 to C16, C11 to C2, C13 to C3, C12 to C4, C7 to C5, C4 to C6, C2 to C7, C1 to C8, C14 to C9, D1 to D2, D6 to D3, H2 to H1, H3 to H2, H1 to H3, L4 to L1, R30 to R1, R1 to R10, R2 to R11, R35 to R12, R15 to R13, R18 to R14, R19 to R15, R32 to R16, R11 to R17, R10 to R18, R31 to R19, R4 to R2, R21 to R20, R17 to R21, R16 to R22, R26 to R28, R34 to R29, R5 to R3, R6 to R4, R29 to R5, R33 to R6, R3 to R9, SW2 to SW1, SW1 to SW2, TP2 to TP1, TP1 to TP2, U4 to U1, U2 to U3, U8 to U4, U6 to U5, U7 to U6, U5 to U7
Routing:
- net GND: track 1.45 -> 14.0 mm
- net /VBUS: track 44.4 -> 51.2 mm
- net +3.3V: track 1.02 -> 6.96 mm
- net /P1.12: track 44.6 -> 49.7 mm
- net /DISPON: track 52.0 -> 56.6 mm
- net /P1.15: track 36.8 -> 41.1 mm
- net /HK-A0: track 9.54 -> 12.4 mm
- net /VBAT: track 55.0 -> 57.8 mm
- net /P1.14: track 39.7 -> 42.5 mm
- net /HK-A1: track 8.26 -> 10.8 mm
- net /AIN0: track 32.8 -> 30.3 mm
- net Net-(U1-X): track 17.4 -> 19.9 mm
- net /HK-A2: track 7.89 -> 10.2 mm
- net /SCL: track 48.5 -> 46.2 mm
- net /PSMODE: track 48.2 -> 50.4 mm
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Other:
- board text added: "ZED Board CPU1-nRF5340 UBlox NORA Rev 1"
- board text removed: "ZED Board CPU1-nRF5340 Rev 1"
